File: pcb/IO_LINK.kicad_pcb (KiCad board)
At the start: 4 copper layers, 120 x 100 mm, 173 parts, among them J1 Screw_Terminal_01x02, J2 USB_B_Mini, J3 STM_PROGRAMING_CONNECTOR, J4 Screw_Terminal_01x04, J5 Screw_Terminal_01x04, J6 Screw_Terminal_01x04, J7 Screw_Terminal_01x04, M1 W5500_ETHERNET_PCB_MODULE, M2 DC_DC_CONVERTER_LM2596_PCB_MO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, SW1 Tactile_Switch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

Commit message: Update Libs for PCb
Parts:
- removed JP3: JUMPER_0805, IO_LINK_LIB:R_0805_2012Metric_Pad1.20x1.40mm_HandSolder
- D18: value SPT01-335DEE -> QFN_3X3_6+3LEAD_STM
Routing:
- net (no net): track 0.00 -> 5.21 mm
- net T3_UC_IRQ: vias 3 -> 2
- net MOSI: vias 2 -> 1
- net GND: vias 464 -> 460
- net G: vias 286 -> 290

Commit message: PCB Release
Parts:
- D18: value QFN_3X3_6+3LEAD_STM -> SPT01-335DEE
- moved C17 9.78 mm to (142.6, 68.2), turned to 90 degrees
- moved M1 5.56 mm to (138.9, 71.7), turned to 0 degrees
Routing:
- net INT_ETH: track 96.8 -> 59.9 mm, vias 2 -> 1
- net CS_ETH: track 84.6 -> 59.2 mm
- net SCLK: track 80.5 -> 60.7 mm
- net MOSI: track 75.5 -> 61.4 mm
- net MISO: track 66.0 -> 76.9 mm
- net 3V3: track 120.6 -> 130.0 mm, vias 38 -> 39
- net RST_ETH: track 74.4 -> 83.2 mm, vias 2 -> 1
- net G: vias 290 -> 288
Other:
- board text added: "Drawn by SFo"
- board text added: "IO_LINK_MASTER HW 0.1"
- board text added: "https://ucandevices.github.io/"
