File: pcb/IO_LINK.sch (KiCad schematic (older format))
At the start: 4 parts

Commit message: PCB Release
Parts:
- H1, H2, H3, H4: symbol IO_LINK_LIB:MountingHole -> IO_LINK-rescue:MountingHole-IO_LINK_LIB
Changed lines of the file:
@@
 EESchema Schematic File Version 4
+LIBS:IO_LINK-cache
 EELAYER 30 0
 EELAYER END
@@
 22.01.2021\n
 $Comp
-L IO_LINK_LIB:MountingHole H1
+L IO_LINK-rescue:MountingHole-IO_LINK_LIB H1
 U 1 1 62AD8F26
 P 700 7550
@@
 $EndComp
 $Comp
-L IO_LINK_LIB:MountingHole H2
+L IO_LINK-rescue:MountingHole-IO_LINK_LIB H2
 U 1 1 62AD96D2
 P 900 7550
@@
 $EndComp
 $Comp
-L IO_LINK_LIB:MountingHole H3
+L IO_LINK-rescue:MountingHole-IO_LINK_LIB H3
 U 1 1 62AD9A2E
 P 1100 7550
@@
 $EndComp
 $Comp
-L IO_LINK_LIB:MountingHole H4
+L IO_LINK-rescue:MountingHole-IO_LINK_LIB H4
 U 1 1 62AD9D79
 P 1300 7550
