File: pcb/IO_LINK_0.sch (KiCad schematic (older format))
At the start: 31 parts, among them J4 Screw_Terminal_01x04, U2 L6360TR

Commit message: PCB Release
Parts:
- C19, C20, C21, C22: symbol IO_LINK_LIB:22pF_50V_0603 -> IO_LINK-rescue:22pF_50V_0603-IO_LINK_LIB
- C23: symbol IO_LINK_LIB:2.2uF_16V_0603 -> IO_LINK-rescue:2.2uF_16V_0603-IO_LINK_LIB
- C24, C28, C30: symbol IO_LINK_LIB:100nF_25V_0603 -> IO_LINK-rescue:100nF_25V_0603-IO_LINK_LIB
- C25: symbol IO_LINK_LIB:10uF_50V_6.3mm_x_5.8mm_electrolytic -> IO_LINK-rescue:10uF_50V_6.3mm_x_5.8mm_electrolytic-IO_LINK_LIB
- C26, C27, C75: symbol IO_LINK_LIB:100nF_50V_0603 -> IO_LINK-rescue:100nF_50V_0603-IO_LINK_LIB
- C29: symbol IO_LINK_LIB:1uF_10V_0603 -> IO_LINK-rescue:1uF_10V_0603-IO_LINK_LIB
- C31, C32: symbol IO_LINK_LIB:560pF_50V_0603 -> IO_LINK-rescue:560pF_50V_0603-IO_LINK_LIB
- D4, D5: symbol IO_LINK_LIB:STPS1L40M -> IO_LINK-rescue:STPS1L40M-IO_LINK_LIB
- D6: symbol IO_LINK_LIB:LED_RED -> IO_LINK-rescue:LED_RED-IO_LINK_LIB
- D7: symbol IO_LINK_LIB:LED_GREEN -> IO_LINK-rescue:LED_GREEN-IO_LINK_LIB
- D8: symbol IO_LINK_LIB:SPT01-335DEE -> IO_LINK-rescue:SPT01-335DEE-IO_LINK_LIB
- J4: symbol IO_LINK_LIB:Screw_Terminal_01x04 -> IO_LINK-rescue:Screw_Terminal_01x04-IO_LINK_LIB
- R10, R11, R12, R9: symbol IO_LINK_LIB:10k_1%_0.1W_0603 -> IO_LINK-rescue:10k_1%_0.1W_0603-IO_LINK_LIB
- R13: symbol IO_LINK_LIB:124k_0.1%_0.1W_0603 -> IO_LINK-rescue:124k_0.1%_0.1W_0603-IO_LINK_LIB
- R14, R15: symbol IO_LINK_LIB:680R_1%_0.1W_0603 -> IO_LINK-rescue:680R_1%_0.1W_0603-IO_LINK_LIB
- R16: symbol IO_LINK_LIB:100R_1%_0.1W_0603 -> IO_LINK-rescue:100R_1%_0.1W_0603-IO_LINK_LIB
- R17: symbol IO_LINK_LIB:15R_1%_0.1W_0603 -> IO_LINK-rescue:15R_1%_0.1W_0603-IO_LINK_LIB
- U2: symbol IO_LINK_LIB:L6360TR -> IO_LINK-rescue:L6360TR-IO_LINK_LIB
Changed lines of the file:
@@
 EESchema Schematic File Version 4
+LIBS:IO_LINK-cache
 EELAYER 30 0
 EELAYER END
@@
 $EndDescr
 $Comp
-L IO_LINK_LIB:L6360TR U?
+L IO_LINK-rescue:L6360TR-IO_LINK_LIB U?
 U 1 1 61DCB27A
 P 8800 4000
@@
 $EndComp
 $Comp
-L IO_LINK_LIB:Screw_Terminal_01x04 J?
+L IO_LINK-rescue:Screw_Terminal_01x04-IO_LINK_LIB J?
 U 1 1 61DCB282
 P 14650 3800
@@
 	9050 5450 9100 5450
 $Comp
-L IO_LINK_LIB:G #PWR?
+L IO_LINK-rescue:G-IO_LINK_LIB #PWR?
 U 1 1 61DCB294
 P 14350 4750
@@
 	14450 4000 14050 4000
 $Comp
-L IO_LINK_LIB:SPT01-335DEE D?
+L IO_LINK-rescue:SPT01-335DEE-IO_LINK_LIB D?
 U 1 1 61DCB2A5
 P 13750 5650
@@
 	14350 3800 14350 4750
 $Comp
-L IO_LINK_LIB:100R_1%_0.1W_0603 R?
+L IO_LINK-rescue:100R_1%_0.1W_0603-IO_LINK_LIB R?
 U 1 1 61DCB2C8
 P 11450 4100
 AR Path="/602CF7CD/61DCB2C8" Ref="R?"  Part="1"
 AR Path="/61D13B0C/61DCB2C8" Ref="R16"  Part="1"
+AR Path="/61DCB2C8" Ref="R16"  Part="1"
 F 0 "R16" V 11350 4100 50  0000 C CNN
 F 1 "100R_1%_0.1W_0603" V 10910 4220 50  0001 C CNN
@@
 $EndComp
 $Comp
-L IO_LINK_LIB:15R_1%_0.1W_0603 R?
+L IO_LINK-rescue:15R_1%_0.1W_0603-IO_LINK_LIB R?
 U 1 1 61DCB2D4
 P 11450 4350
@@
 $EndComp
 $Comp
-L IO_LINK_LIB:STPS1L40M D?
+L IO_LINK-rescue:STPS1L40M-IO_LINK_LIB D?
 U 1 1 61DCB2DD
 P 10350 4400
@@
 $EndComp
 $Comp
-L IO_LINK_LIB:560pF_50V_0603 C?
+L IO_LINK-rescue:560pF_50V_0603-IO_LINK_LIB C?
 U 1 1 61DCB2E8
 P 12650 4400
@@
 $EndComp
 $Comp
-L IO_LINK_LIB:10uF_50V_6.3mm_x_5.8mm_electrolytic C?
+L IO_LINK-rescue:10uF_50V_6.3mm_x_5.8mm_electrolytic-IO_LINK_LIB C?
 U 1 1 61DCB2F3
 P 7000 2000
@@
 $EndComp
 $Comp
-L IO_LINK_LIB:100nF_50V_0603 C?
+L IO_LINK-rescue:100nF_50V_0603-IO_LINK_LIB C?
 U 1 1 61DCB2FE
 P 7950 2000
@@
 	10350 4000 10350 4250
 $Comp
-L IO_LINK_LIB:STPS1L40M D?
+L IO_LINK-rescue:STPS1L40M-IO_LINK_LIB D?
 U 1 1 61DCB31C
 P 10700 4400
@@
 	13150 4550 13150 4750
 $Comp
-L IO_LINK_LIB:560pF_50V_0603 C?
+L IO_LINK-rescue:560pF_50V_0603-IO_LINK_LIB C?
 U 1 1 61DCB354
 P 13150 4400
@@
 	9800 4550 10000 4550
 $Comp
-L IO_LINK_LIB:680R_1%_0.1W_0603 R?
+L IO_LINK-rescue:680R_1%_0.1W_0603-IO_LINK_LIB R?
 U 1 1 61DCB39E
 P 10600 5200
@@
 	10000 4550 10000 5200
 $Comp
-L IO_LINK_LIB:680R_1%_0.1W_0603 R?
+L IO_LINK-rescue:680R_1%_0.1W_0603-IO_LINK_LIB R?
 U 1 1 61DCB3AC
 P 10600 5500
@@
 $EndComp
 $Comp
-L IO_LINK_LIB:LED_RED D?
+L IO_LINK-rescue:LED_RED-IO_LINK_LIB D?
 U 1 1 61DCB3B6
 P 11500 5200
@@
 $EndComp
 $Comp
-L IO_LINK_LIB:LED_GREEN D?
+L IO_LINK-rescue:LED_GREEN-IO_LINK_LIB D?
 U 1 1 61DCB3C0
 P 11500 5500
@@
 	11900 5350 11900 5200
 $Comp
-L IO_LINK_LIB:3V3_T0 #PWR?
+L IO_LINK-rescue:3V3_T0-IO_LINK_LIB #PWR?
 U 1 1 61DCB3CF
 P 12150 5250
@@
 	11900 5350 12150 5350
 $Comp
-L IO_LINK_LIB:100nF_25V_0603 C?
+L IO_LINK-rescue:100nF_25V_0603-IO_LINK_LIB C?
 U 1 1 61DCB3DC
 P 10450 3350
@@
 	9800 3350 10000 3350
 $Comp
-L IO_LINK_LIB:3V3_T0 #PWR?
+L IO_LINK-rescue:3V3_T0-IO_LINK_LIB #PWR?
 U 1 1 61DCB3EB
 P 10000 3200
@@
 	10000 3350 10300 3350
 $Comp
-L IO_LINK_LIB:100nF_25V_0603 C?
+L IO_LINK-rescue:100nF_25V_0603-IO_LINK_LIB C?
 U 1 1 61DCB3F9
 P 9750 2000
@@
 	9750 2150 9750 2350
 $Comp
-L IO_LINK_LIB:100nF_50V_0603 C?
+L IO_LINK-rescue:100nF_50V_0603-IO_LINK_LIB C?
 U 1 1 61DCB40B
 P 7450 2000
@@
 	7000 2150 7000 2350
 $Comp
-L IO_LINK_LIB:VCC #PWR?
+L IO_LINK-rescue:VCC-IO_LINK_LIB #PWR?
 U 1 1 61DCB428
 P 7300 1750
@@
 $EndComp
 $Comp
-L IO_LINK_LIB:VCC #PWR?
+L IO_LINK-rescue:VCC-IO_LINK_LIB #PWR?
 U 1 1 61DCB42E
 P 7800 1750
@@
 	7450 1800 7450 1850
 $Comp
-L IO_LINK_LIB:VCC #PWR?
+L IO_LINK-rescue:VCC-IO_LINK_LIB #PWR?
 U 1 1 61DCB43B
 P 7000 1750
@@
 	8600 1550 7450 1550
 $Comp
-L IO_LINK_LIB:2.2uF_16V_0603 C?
+L IO_LINK-rescue:2.2uF_16V_0603-IO_LINK_LIB C?
 U 1 1 61DCB44A
 P 5700 2000
@@
 $EndComp
 $Comp
-L IO_LINK_LIB:100nF_25V_0603 C?
+L IO_LINK-rescue:100nF_25V_0603-IO_LINK_LIB C?
 U 1 1 61DCB455
 P 6200 2000
@@
 Connection ~ 5700 1550
 $Comp
-L IO_LINK_LIB:8V #PWR?
+L IO_LINK-rescue:8V-IO_LINK_LIB #PWR?
 U 1 1 61DCB471
 P 5600 1500
@@
 	5600 1500 5600 1550
 $Comp
-L IO_LINK_LIB:1uF_10V_0603 C?
+L IO_LINK-rescue:1uF_10V_0603-IO_LINK_LIB C?
 U 1 1 61DCB47D
 P 10250 2000
@@
 Connection ~ 10250 1550
 $Comp
-L IO_LINK_LIB:3V3_T0 #PWR?
+L IO_LINK-rescue:3V3_T0-IO_LINK_LIB #PWR?
 U 1 1 61DCB492
 P 10350 1500
@@
 	4800 3350 7800 3350
 $Comp
-L IO_LINK_LIB:10k_1%_0.1W_0603 R?
+L IO_LINK-rescue:10k_1%_0.1W_0603-IO_LINK_LIB R?
 U 1 1 61DCB49F
 P 4800 2900
@@
 	4800 3050 4800 3350
 $Comp
-L IO_LINK_LIB:10k_1%_0.1W_0603 R?
+L IO_LINK-rescue:10k_1%_0.1W_0603-IO_LINK_LIB R?
 U 1 1 61DCB4AC
 P 4300 2900
@@
 	4300 3450 4300 3050
 $Comp
-L IO_LINK_LIB:10k_1%_0.1W_0603 R?
+L IO_LINK-rescue:10k_1%_0.1W_0603-IO_LINK_LIB R?
 U 1 1 61DCB4B9
 P 3800 2900
@@
 	3800 3550 3800 3050
 $Comp
-L IO_LINK_LIB:10k_1%_0.1W_0603 R?
+L IO_LINK-rescue:10k_1%_0.1W_0603-IO_LINK_LIB R?
 U 1 1 61DCB4C6
 P 3300 2900
@@
 	3300 3650 3300 3050
 $Comp
-L IO_LINK_LIB:3V3 #PWR?
+L IO_LINK-rescue:3V3-IO_LINK_LIB #PWR?
 U 1 1 61DCB4CD
 P 3300 2550
@@
 $EndComp
 $Comp
-L IO_LINK_LIB:3V3 #PWR?
+L IO_LINK-rescue:3V3-IO_LINK_LIB #PWR?
 U 1 1 61DCB4D3
 P 3800 2550
@@
 $EndComp
 $Comp
-L IO_LINK_LIB:3V3 #PWR?
+L IO_LINK-rescue:3V3-IO_LINK_LIB #PWR?
 U 1 1 61DCB4D9
 P 4300 2550
@@
 $EndComp
 $Comp
-L IO_LINK_LIB:3V3 #PWR?
+L IO_LINK-rescue:3V3-IO_LINK_LIB #PWR?
 U 1 1 61DCB4DF
 P 4800 2550
@@
 	3300 2550 3300 2750
 $Comp
-L IO_LINK_LIB:22pF_50V_0603 C?
+L IO_LINK-rescue:22pF_50V_0603-IO_LINK_LIB C?
 U 1 1 61DCB4EE
 P 3800 4100
@@
 $EndComp
 $Comp
-L IO_LINK_LIB:22pF_50V_0603 C?
+L IO_LINK-rescue:22pF_50V_0603-IO_LINK_LIB C?
 U 1 1 61DCB4F9
 P 4800 4100
@@
 $EndComp
 $Comp
-L IO_LINK_LIB:22pF_50V_0603 C?
+L IO_LINK-rescue:22pF_50V_0603-IO_LINK_LIB C?
 U 1 1 61DCB504
 P 4300 4100
@@
 $EndComp
 $Comp
-L IO_LINK_LIB:22pF_50V_0603 C?
+L IO_LINK-rescue:22pF_50V_0603-IO_LINK_LIB C?
 U 1 1 61DCB50F
 P 3300 4100
@@
 T0_UC_SIO
 $Comp
-L IO_LINK_LIB:124k_0.1%_0.1W_0603 R?
+L IO_LINK-rescue:124k_0.1%_0.1W_0603-IO_LINK_LIB R?
 U 1 1 61DCB550
 P 8050 5450
@@
 	11900 4000 13150 4000
 $Comp
-L IO_LINK_LIB:100nF_50V_0603 C?
+L IO_LINK-rescue:100nF_50V_0603-IO_LINK_LIB C?
 U 1 1 606822AA
 P 12150 4400
