File: pcb/IO_LINK_1.sch (KiCad schematic (older format))
At the start: 31 parts, among them J5 Screw_Terminal_01x04, U3 L6360TR

Commit message: PCB Release
Parts:
- C33, C34, C35, C36: symbol IO_LINK_LIB:22pF_50V_0603 -> IO_LINK-rescue:22pF_50V_0603-IO_LINK_LIB
- C37: symbol IO_LINK_LIB:2.2uF_16V_0603 -> IO_LINK-rescue:2.2uF_16V_0603-IO_LINK_LIB
- C38, C42, C44: symbol IO_LINK_LIB:100nF_25V_0603 -> IO_LINK-rescue:100nF_25V_0603-IO_LINK_LIB
- C39: symbol IO_LINK_LIB:10uF_50V_6.3mm_x_5.8mm_electrolytic -> IO_LINK-rescue:10uF_50V_6.3mm_x_5.8mm_electrolytic-IO_LINK_LIB
- C40, C41, C76: symbol IO_LINK_LIB:100nF_50V_0603 -> IO_LINK-rescue:100nF_50V_0603-IO_LINK_LIB
- C43: symbol IO_LINK_LIB:1uF_10V_0603 -> IO_LINK-rescue:1uF_10V_0603-IO_LINK_LIB
- C45, C46: symbol IO_LINK_LIB:560pF_50V_0603 -> IO_LINK-rescue:560pF_50V_0603-IO_LINK_LIB
- D10, D9: symbol IO_LINK_LIB:STPS1L40M -> IO_LINK-rescue:STPS1L40M-IO_LINK_LIB
- D11: symbol IO_LINK_LIB:LED_RED -> IO_LINK-rescue:LED_RED-IO_LINK_LIB
- D12: symbol IO_LINK_LIB:LED_GREEN -> IO_LINK-rescue:LED_GREEN-IO_LINK_LIB
- D13: symbol IO_LINK_LIB:SPT01-335DEE -> IO_LINK-rescue:SPT01-335DEE-IO_LINK_LIB
- J5: symbol IO_LINK_LIB:Screw_Terminal_01x04 -> IO_LINK-rescue:Screw_Terminal_01x04-IO_LINK_LIB
- R18, R19, R20, R21: symbol IO_LINK_LIB:10k_1%_0.1W_0603 -> IO_LINK-rescue:10k_1%_0.1W_0603-IO_LINK_LIB
- R22: symbol IO_LINK_LIB:124k_0.1%_0.1W_0603 -> IO_LINK-rescue:124k_0.1%_0.1W_0603-IO_LINK_LIB
- R23, R24: symbol IO_LINK_LIB:680R_1%_0.1W_0603 -> IO_LINK-rescue:680R_1%_0.1W_0603-IO_LINK_LIB
- R25: symbol IO_LINK_LIB:100R_1%_0.1W_0603 -> IO_LINK-rescue:100R_1%_0.1W_0603-IO_LINK_LIB
- R26: symbol IO_LINK_LIB:15R_1%_0.1W_0603 -> IO_LINK-rescue:15R_1%_0.1W_0603-IO_LINK_LIB
- U3: symbol IO_LINK_LIB:L6360TR -> IO_LINK-rescue:L6360TR-IO_LINK_LIB
Changed lines of the file:
@@
 EESchema Schematic File Version 4
+LIBS:IO_LINK-cache
 EELAYER 30 0
 EELAYER END
@@
 $EndDescr
 $Comp
-L IO_LINK_LIB:L6360TR U?
+L IO_LINK-rescue:L6360TR-IO_LINK_LIB U?
 U 1 1 61E63877
 P 8800 4100
@@
 $EndComp
 $Comp
-L IO_LINK_LIB:Screw_Terminal_01x04 J?
+L IO_LINK-rescue:Screw_Terminal_01x04-IO_LINK_LIB J?
 U 1 1 61E6387F
 P 14650 3900
@@
 	9050 5550 9100 5550
 $Comp
-L IO_LINK_LIB:G #PWR?
+L IO_LINK-rescue:G-IO_LINK_LIB #PWR?
 U 1 1 61E63891
 P 14350 4850
@@
 	14450 4100 14050 4100
 $Comp
-L IO_LINK_LIB:SPT01-335DEE D?
+L IO_LINK-rescue:SPT01-335DEE-IO_LINK_LIB D?
 U 1 1 61E638A2
 P 13750 5750
@@
 	14350 3900 14350 4850
 $Comp
-L IO_LINK_LIB:100R_1%_0.1W_0603 R?
+L IO_LINK-rescue:100R_1%_0.1W_0603-IO_LINK_LIB R?
 U 1 1 61E638C5
 P 11450 4200
 AR Path="/602CF7CD/61E638C5" Ref="R?"  Part="1"
 AR Path="/61DF74C5/61E638C5" Ref="R25"  Part="1"
+AR Path="/61E638C5" Ref="R25"  Part="1"
 F 0 "R25" V 11350 4200 50  0000 C CNN
 F 1 "100R_1%_0.1W_0603" V 10910 4320 50  0001 C CNN
@@
 $EndComp
 $Comp
-L IO_LINK_LIB:15R_1%_0.1W_0603 R?
+L IO_LINK-rescue:15R_1%_0.1W_0603-IO_LINK_LIB R?
 U 1 1 61E638D1
 P 11450 4450
@@
 $EndComp
 $Comp
-L IO_LINK_LIB:STPS1L40M D?
+L IO_LINK-rescue:STPS1L40M-IO_LINK_LIB D?
 U 1 1 61E638DA
 P 10350 4500
@@
 $EndComp
 $Comp
-L IO_LINK_LIB:10uF_50V_6.3mm_x_5.8mm_electrolytic C?
+L IO_LINK-rescue:10uF_50V_6.3mm_x_5.8mm_electrolytic-IO_LINK_LIB C?
 U 1 1 61E638F0
 P 7000 2100
@@
 $EndComp
 $Comp
-L IO_LINK_LIB:100nF_50V_0603 C?
+L IO_LINK-rescue:100nF_50V_0603-IO_LINK_LIB C?
 U 1 1 61E638FB
 P 7950 2100
@@
 	10350 4100 10350 4350
 $Comp
-L IO_LINK_LIB:STPS1L40M D?
+L IO_LINK-rescue:STPS1L40M-IO_LINK_LIB D?
 U 1 1 61E63919
 P 10700 4500
@@
 	9800 4650 10000 4650
 $Comp
-L IO_LINK_LIB:680R_1%_0.1W_0603 R?
+L IO_LINK-rescue:680R_1%_0.1W_0603-IO_LINK_LIB R?
 U 1 1 61E6399B
 P 10600 5300
@@
 	10000 4650 10000 5300
 $Comp
-L IO_LINK_LIB:680R_1%_0.1W_0603 R?
+L IO_LINK-rescue:680R_1%_0.1W_0603-IO_LINK_LIB R?
 U 1 1 61E639A9
 P 10600 5600
@@
 $EndComp
 $Comp
-L IO_LINK_LIB:LED_RED D?
+L IO_LINK-rescue:LED_RED-IO_LINK_LIB D?
 U 1 1 61E639B3
 P 11500 5300
@@
 $EndComp
 $Comp
-L IO_LINK_LIB:LED_GREEN D?
+L IO_LINK-rescue:LED_GREEN-IO_LINK_LIB D?
 U 1 1 61E639BD
 P 11500 5600
@@
 	11900 5450 12150 5450
 $Comp
-L IO_LINK_LIB:100nF_25V_0603 C?
+L IO_LINK-rescue:100nF_25V_0603-IO_LINK_LIB C?
 U 1 1 61E639D3
 P 10450 3450
@@
 	10000 3450 10300 3450
 $Comp
-L IO_LINK_LIB:100nF_25V_0603 C?
+L IO_LINK-rescue:100nF_25V_0603-IO_LINK_LIB C?
 U 1 1 61E639EA
 P 9750 2100
@@
 	9750 2250 9750 2450
 $Comp
-L IO_LINK_LIB:100nF_50V_0603 C?
+L IO_LINK-rescue:100nF_50V_0603-IO_LINK_LIB C?
 U 1 1 61E639FC
 P 7450 2100
@@
 	7000 2250 7000 2450
 $Comp
-L IO_LINK_LIB:VCC #PWR?
+L IO_LINK-rescue:VCC-IO_LINK_LIB #PWR?
 U 1 1 61E63A19
 P 7300 1850
@@
 $EndComp
 $Comp
-L IO_LINK_LIB:VCC #PWR?
+L IO_LINK-rescue:VCC-IO_LINK_LIB #PWR?
 U 1 1 61E63A1F
 P 7800 1850
@@
 	7450 1900 7450 1950
 $Comp
-L IO_LINK_LIB:VCC #PWR?
+L IO_LINK-rescue:VCC-IO_LINK_LIB #PWR?
 U 1 1 61E63A2C
 P 7000 1850
@@
 	8600 1650 7450 1650
 $Comp
-L IO_LINK_LIB:2.2uF_16V_0603 C?
+L IO_LINK-rescue:2.2uF_16V_0603-IO_LINK_LIB C?
 U 1 1 61E63A3B
 P 5700 2100
@@
 $EndComp
 $Comp
-L IO_LINK_LIB:100nF_25V_0603 C?
+L IO_LINK-rescue:100nF_25V_0603-IO_LINK_LIB C?
 U 1 1 61E63A46
 P 6200 2100
@@
 Connection ~ 5700 1650
 $Comp
-L IO_LINK_LIB:8V #PWR?
+L IO_LINK-rescue:8V-IO_LINK_LIB #PWR?
 U 1 1 61E63A62
 P 5600 1600
@@
 	5600 1600 5600 1650
 $Comp
-L IO_LINK_LIB:1uF_10V_0603 C?
+L IO_LINK-rescue:1uF_10V_0603-IO_LINK_LIB C?
 U 1 1 61E63A6E
 P 10250 2100
@@
 	4800 3450 7800 3450
 $Comp
-L IO_LINK_LIB:10k_1%_0.1W_0603 R?
+L IO_LINK-rescue:10k_1%_0.1W_0603-IO_LINK_LIB R?
 U 1 1 61E63A8A
 P 4800 3000
@@
 	4800 3150 4800 3450
 $Comp
-L IO_LINK_LIB:10k_1%_0.1W_0603 R?
+L IO_LINK-rescue:10k_1%_0.1W_0603-IO_LINK_LIB R?
 U 1 1 61E63A97
 P 4300 3000
@@
 	4300 3550 4300 3150
 $Comp
-L IO_LINK_LIB:10k_1%_0.1W_0603 R?
+L IO_LINK-rescue:10k_1%_0.1W_0603-IO_LINK_LIB R?
 U 1 1 61E63AA4
 P 3800 3000
@@
 	3800 3650 3800 3150
 $Comp
-L IO_LINK_LIB:10k_1%_0.1W_0603 R?
+L IO_LINK-rescue:10k_1%_0.1W_0603-IO_LINK_LIB R?
 U 1 1 61E63AB1
 P 3300 3000
@@
 	3300 3750 3300 3150
 $Comp
-L IO_LINK_LIB:3V3 #PWR?
+L IO_LINK-rescue:3V3-IO_LINK_LIB #PWR?
 U 1 1 61E63AB8
 P 3300 2650
@@
 $EndComp
 $Comp
-L IO_LINK_LIB:3V3 #PWR?
+L IO_LINK-rescue:3V3-IO_LINK_LIB #PWR?
 U 1 1 61E63ABE
 P 3800 2650
@@
 $EndComp
 $Comp
-L IO_LINK_LIB:3V3 #PWR?
+L IO_LINK-rescue:3V3-IO_LINK_LIB #PWR?
 U 1 1 61E63AC4
 P 4300 2650
@@
 $EndComp
 $Comp
-L IO_LINK_LIB:3V3 #PWR?
+L IO_LINK-rescue:3V3-IO_LINK_LIB #PWR?
 U 1 1 61E63ACA
 P 4800 2650
@@
 	3300 2650 3300 2850
 $Comp
-L IO_LINK_LIB:22pF_50V_0603 C?
+L IO_LINK-rescue:22pF_50V_0603-IO_LINK_LIB C?
 U 1 1 61E63AD9
 P 3800 4200
@@
 $EndComp
 $Comp
-L IO_LINK_LIB:22pF_50V_0603 C?
+L IO_LINK-rescue:22pF_50V_0603-IO_LINK_LIB C?
 U 1 1 61E63AE4
 P 4800 4200
@@
 $EndComp
 $Comp
-L IO_LINK_LIB:22pF_50V_0603 C?
+L IO_LINK-rescue:22pF_50V_0603-IO_LINK_LIB C?
 U 1 1 61E63AEF
 P 4300 4200
@@
 $EndComp
 $Comp
-L IO_LINK_LIB:22pF_50V_0603 C?
+L IO_LINK-rescue:22pF_50V_0603-IO_LINK_LIB C?
 U 1 1 61E63AFA
 P 3300 4200
@@
 T1_UC_SIO
 $Comp
-L IO_LINK_LIB:124k_0.1%_0.1W_0603 R?
+L IO_LINK-rescue:124k_0.1%_0.1W_0603-IO_LINK_LIB R?
 U 1 1 61E63B3B
 P 8050 5550
@@
 IO-LINK TRANSCEIVER no. 1\n
 $Comp
-L IO_LINK_LIB:3V3_T1 #PWR?
+L IO_LINK-rescue:3V3_T1-IO_LINK_LIB #PWR?
 U 1 1 61E63B59
 P 10350 1600
@@
 $EndComp
 $Comp
-L IO_LINK_LIB:3V3_T1 #PWR?
+L IO_LINK-rescue:3V3_T1-IO_LINK_LIB #PWR?
 U 1 1 61E63B5F
 P 10000 3300
@@
 $EndComp
 $Comp
-L IO_LINK_LIB:3V3_T1 #PWR?
+L IO_LINK-rescue:3V3_T1-IO_LINK_LIB #PWR?
 U 1 1 61E63B65
 P 12150 5350
@@
 	7800 4350 7250 4350
 $Comp
-L IO_LINK_LIB:3V3_T1 #PWR?
+L IO_LINK-rescue:3V3_T1-IO_LINK_LIB #PWR?
 U 1 1 604AA647
 P 6700 4450
@@
 	9800 3900 12150 3900
 $Comp
-L IO_LINK_LIB:560pF_50V_0603 C?
+L IO_LINK-rescue:560pF_50V_0603-IO_LINK_LIB C?
 U 1 1 61E63951
 P 13100 4500
@@
 	12600 4650 12600 4850
 $Comp
-L IO_LINK_LIB:560pF_50V_0603 C?
+L IO_LINK-rescue:560pF_50V_0603-IO_LINK_LIB C?
 U 1 1 61E638E5
 P 12600 4500
@@
 	12600 4000 12600 4350
 $Comp
-L IO_LINK_LIB:100nF_50V_0603 C?
+L IO_LINK-rescue:100nF_50V_0603-IO_LINK_LIB C?
 U 1 1 606C50E5
 P 12150 4500
