File: pcb/IO_LINK_2.sch (KiCad schematic (older format))
At the start: 31 parts, among them J6 Screw_Terminal_01x04, U4 L6360TR

Commit message: PCB Release
Parts:
- C47, C48, C49, C50: symbol IO_LINK_LIB:22pF_50V_0603 -> IO_LINK-rescue:22pF_50V_0603-IO_LINK_LIB
- C51: symbol IO_LINK_LIB:2.2uF_16V_0603 -> IO_LINK-rescue:2.2uF_16V_0603-IO_LINK_LIB
- C52, C56, C58: symbol IO_LINK_LIB:100nF_25V_0603 -> IO_LINK-rescue:100nF_25V_0603-IO_LINK_LIB
- C53: symbol IO_LINK_LIB:10uF_50V_6.3mm_x_5.8mm_electrolytic -> IO_LINK-rescue:10uF_50V_6.3mm_x_5.8mm_electrolytic-IO_LINK_LIB
- C54, C55, C77: symbol IO_LINK_LIB:100nF_50V_0603 -> IO_LINK-rescue:100nF_50V_0603-IO_LINK_LIB
- C57: symbol IO_LINK_LIB:1uF_10V_0603 -> IO_LINK-rescue:1uF_10V_0603-IO_LINK_LIB
- C59, C60: symbol IO_LINK_LIB:560pF_50V_0603 -> IO_LINK-rescue:560pF_50V_0603-IO_LINK_LIB
- D14, D15: symbol IO_LINK_LIB:STPS1L40M -> IO_LINK-rescue:STPS1L40M-IO_LINK_LIB
- D16: symbol IO_LINK_LIB:LED_RED -> IO_LINK-rescue:LED_RED-IO_LINK_LIB
- D17: symbol IO_LINK_LIB:LED_GREEN -> IO_LINK-rescue:LED_GREEN-IO_LINK_LIB
- D18: symbol IO_LINK_LIB:SPT01-335DEE -> IO_LINK-rescue:SPT01-335DEE-IO_LINK_LIB
- J6: symbol IO_LINK_LIB:Screw_Terminal_01x04 -> IO_LINK-rescue:Screw_Terminal_01x04-IO_LINK_LIB
- R27, R28, R29, R30: symbol IO_LINK_LIB:10k_1%_0.1W_0603 -> IO_LINK-rescue:10k_1%_0.1W_0603-IO_LINK_LIB
- R31: symbol IO_LINK_LIB:124k_0.1%_0.1W_0603 -> IO_LINK-rescue:124k_0.1%_0.1W_0603-IO_LINK_LIB
- R32, R33: symbol IO_LINK_LIB:680R_1%_0.1W_0603 -> IO_LINK-rescue:680R_1%_0.1W_0603-IO_LINK_LIB
- R34: symbol IO_LINK_LIB:100R_1%_0.1W_0603 -> IO_LINK-rescue:100R_1%_0.1W_0603-IO_LINK_LIB
- R35: symbol IO_LINK_LIB:15R_1%_0.1W_0603 -> IO_LINK-rescue:15R_1%_0.1W_0603-IO_LINK_LIB
- U4: symbol IO_LINK_LIB:L6360TR -> IO_LINK-rescue:L6360TR-IO_LINK_LIB
Changed lines of the file:
@@
 EESchema Schematic File Version 4
+LIBS:IO_LINK-cache
 EELAYER 30 0
 EELAYER END
@@
 $EndDescr
 $Comp
-L IO_LINK_LIB:L6360TR U?
+L IO_LINK-rescue:L6360TR-IO_LINK_LIB U?
 U 1 1 61EA17D4
 P 8800 4150
@@
 	8600 5500 8600 5700
 $Comp
-L IO_LINK_LIB:100R_1%_0.1W_0603 R?
+L IO_LINK-rescue:100R_1%_0.1W_0603-IO_LINK_LIB R?
 U 1 1 61EA1822
 P 11450 4250
 AR Path="/602CF7CD/61EA1822" Ref="R?"  Part="1"
 AR Path="/61E6C006/61EA1822" Ref="R34"  Part="1"
+AR Path="/61EA1822" Ref="R34"  Part="1"
 F 0 "R34" V 11350 4250 50  0000 C CNN
 F 1 "100R_1%_0.1W_0603" V 10910 4370 50  0001 C CNN
@@
 $EndComp
 $Comp
-L IO_LINK_LIB:15R_1%_0.1W_0603 R?
+L IO_LINK-rescue:15R_1%_0.1W_0603-IO_LINK_LIB R?
 U 1 1 61EA182E
 P 11450 4500
@@
 $EndComp
 $Comp
-L IO_LINK_LIB:STPS1L40M D?
+L IO_LINK-rescue:STPS1L40M-IO_LINK_LIB D?
 U 1 1 61EA1837
 P 10350 4550
@@
 $EndComp
 $Comp
-L IO_LINK_LIB:560pF_50V_0603 C?
+L IO_LINK-rescue:560pF_50V_0603-IO_LINK_LIB C?
 U 1 1 61EA1842
 P 12600 4550
@@
 $EndComp
 $Comp
-L IO_LINK_LIB:10uF_50V_6.3mm_x_5.8mm_electrolytic C?
+L IO_LINK-rescue:10uF_50V_6.3mm_x_5.8mm_electrolytic-IO_LINK_LIB C?
 U 1 1 61EA184D
 P 7000 2150
@@
 $EndComp
 $Comp
-L IO_LINK_LIB:100nF_50V_0603 C?
+L IO_LINK-rescue:100nF_50V_0603-IO_LINK_LIB C?
 U 1 1 61EA1858
 P 7950 2150
@@
 	10350 4150 10350 4400
 $Comp
-L IO_LINK_LIB:STPS1L40M D?
+L IO_LINK-rescue:STPS1L40M-IO_LINK_LIB D?
 U 1 1 61EA1876
 P 10700 4550
@@
 	13100 4700 13100 4900
 $Comp
-L IO_LINK_LIB:560pF_50V_0603 C?
+L IO_LINK-rescue:560pF_50V_0603-IO_LINK_LIB C?
 U 1 1 61EA18AE
 P 13100 4550
@@
 	9800 4700 10000 4700
 $Comp
-L IO_LINK_LIB:680R_1%_0.1W_0603 R?
+L IO_LINK-rescue:680R_1%_0.1W_0603-IO_LINK_LIB R?
 U 1 1 61EA18F8
 P 10600 5350
@@
 	10000 4700 10000 5350
 $Comp
-L IO_LINK_LIB:680R_1%_0.1W_0603 R?
+L IO_LINK-rescue:680R_1%_0.1W_0603-IO_LINK_LIB R?
 U 1 1 61EA1906
 P 10600 5650
@@
 $EndComp
 $Comp
-L IO_LINK_LIB:LED_RED D?
+L IO_LINK-rescue:LED_RED-IO_LINK_LIB D?
 U 1 1 61EA1910
 P 11500 5350
@@
 $EndComp
 $Comp
-L IO_LINK_LIB:LED_GREEN D?
+L IO_LINK-rescue:LED_GREEN-IO_LINK_LIB D?
 U 1 1 61EA191A
 P 11500 5650
@@
 	11900 5500 12150 5500
 $Comp
-L IO_LINK_LIB:100nF_25V_0603 C?
+L IO_LINK-rescue:100nF_25V_0603-IO_LINK_LIB C?
 U 1 1 61EA1930
 P 10450 3500
@@
 	10000 3500 10300 3500
 $Comp
-L IO_LINK_LIB:100nF_25V_0603 C?
+L IO_LINK-rescue:100nF_25V_0603-IO_LINK_LIB C?
 U 1 1 61EA1947
 P 9750 2150
@@
 	9750 2300 9750 2500
 $Comp
-L IO_LINK_LIB:100nF_50V_0603 C?
+L IO_LINK-rescue:100nF_50V_0603-IO_LINK_LIB C?
 U 1 1 61EA1959
 P 7450 2150
@@
 	7000 2300 7000 2500
 $Comp
-L IO_LINK_LIB:VCC #PWR?
+L IO_LINK-rescue:VCC-IO_LINK_LIB #PWR?
 U 1 1 61EA1976
 P 7300 1900
@@
 $EndComp
 $Comp
-L IO_LINK_LIB:VCC #PWR?
+L IO_LINK-rescue:VCC-IO_LINK_LIB #PWR?
 U 1 1 61EA197C
 P 7800 1900
@@
 	7450 1950 7450 2000
 $Comp
-L IO_LINK_LIB:VCC #PWR?
+L IO_LINK-rescue:VCC-IO_LINK_LIB #PWR?
 U 1 1 61EA1989
 P 7000 1900
@@
 	8600 1700 7450 1700
 $Comp
-L IO_LINK_LIB:2.2uF_16V_0603 C?
+L IO_LINK-rescue:2.2uF_16V_0603-IO_LINK_LIB C?
 U 1 1 61EA1998
 P 5700 2150
@@
 $EndComp
 $Comp
-L IO_LINK_LIB:100nF_25V_0603 C?
+L IO_LINK-rescue:100nF_25V_0603-IO_LINK_LIB C?
 U 1 1 61EA19A3
 P 6200 2150
@@
 Connection ~ 5700 1700
 $Comp
-L IO_LINK_LIB:8V #PWR?
+L IO_LINK-rescue:8V-IO_LINK_LIB #PWR?
 U 1 1 61EA19BF
 P 5600 1650
@@
 	5600 1650 5600 1700
 $Comp
-L IO_LINK_LIB:1uF_10V_0603 C?
+L IO_LINK-rescue:1uF_10V_0603-IO_LINK_LIB C?
 U 1 1 61EA19CB
 P 10250 2150
@@
 	4800 3500 7800 3500
 $Comp
-L IO_LINK_LIB:10k_1%_0.1W_0603 R?
+L IO_LINK-rescue:10k_1%_0.1W_0603-IO_LINK_LIB R?
 U 1 1 61EA19E7
 P 4800 3050
@@
 	4800 3200 4800 3500
 $Comp
-L IO_LINK_LIB:10k_1%_0.1W_0603 R?
+L IO_LINK-rescue:10k_1%_0.1W_0603-IO_LINK_LIB R?
 U 1 1 61EA19F4
 P 4300 3050
@@
 	4300 3600 4300 3200
 $Comp
-L IO_LINK_LIB:10k_1%_0.1W_0603 R?
+L IO_LINK-rescue:10k_1%_0.1W_0603-IO_LINK_LIB R?
 U 1 1 61EA1A01
 P 3800 3050
@@
 	3800 3700 3800 3200
 $Comp
-L IO_LINK_LIB:10k_1%_0.1W_0603 R?
+L IO_LINK-rescue:10k_1%_0.1W_0603-IO_LINK_LIB R?
 U 1 1 61EA1A0E
 P 3300 3050
@@
 	3300 3800 3300 3200
 $Comp
-L IO_LINK_LIB:3V3 #PWR?
+L IO_LINK-rescue:3V3-IO_LINK_LIB #PWR?
 U 1 1 61EA1A15
 P 3300 2700
@@
 $EndComp
 $Comp
-L IO_LINK_LIB:3V3 #PWR?
+L IO_LINK-rescue:3V3-IO_LINK_LIB #PWR?
 U 1 1 61EA1A1B
 P 3800 2700
@@
 $EndComp
 $Comp
-L IO_LINK_LIB:3V3 #PWR?
+L IO_LINK-rescue:3V3-IO_LINK_LIB #PWR?
 U 1 1 61EA1A21
 P 4300 2700
@@
 $EndComp
 $Comp
-L IO_LINK_LIB:3V3 #PWR?
+L IO_LINK-rescue:3V3-IO_LINK_LIB #PWR?
 U 1 1 61EA1A27
 P 4800 2700
@@
 	3300 2700 3300 2900
 $Comp
-L IO_LINK_LIB:22pF_50V_0603 C?
+L IO_LINK-rescue:22pF_50V_0603-IO_LINK_LIB C?
 U 1 1 61EA1A36
 P 3800 4250
@@
 $EndComp
 $Comp
-L IO_LINK_LIB:22pF_50V_0603 C?
+L IO_LINK-rescue:22pF_50V_0603-IO_LINK_LIB C?
 U 1 1 61EA1A41
 P 4800 4250
@@
 $EndComp
 $Comp
-L IO_LINK_LIB:22pF_50V_0603 C?
+L IO_LINK-rescue:22pF_50V_0603-IO_LINK_LIB C?
 U 1 1 61EA1A4C
 P 4300 4250
@@
 $EndComp
 $Comp
-L IO_LINK_LIB:22pF_50V_0603 C?
+L IO_LINK-rescue:22pF_50V_0603-IO_LINK_LIB C?
 U 1 1 61EA1A57
 P 3300 4250
@@
 T2_UC_SIO
 $Comp
-L IO_LINK_LIB:124k_0.1%_0.1W_0603 R?
+L IO_LINK-rescue:124k_0.1%_0.1W_0603-IO_LINK_LIB R?
 U 1 1 61EA1A98
 P 8050 5600
@@
 IO-LINK TRANSCEIVER no. 2
 $Comp
-L IO_LINK_LIB:3V3_T2 #PWR?
+L IO_LINK-rescue:3V3_T2-IO_LINK_LIB #PWR?
 U 1 1 61EA1AB6
 P 10350 1650
@@
 $EndComp
 $Comp
-L IO_LINK_LIB:3V3_T2 #PWR?
+L IO_LINK-rescue:3V3_T2-IO_LINK_LIB #PWR?
 U 1 1 61EA1ABC
 P 12150 5400
@@
 $EndComp
 $Comp
-L IO_LINK_LIB:3V3_T2 #PWR?
+L IO_LINK-rescue:3V3_T2-IO_LINK_LIB #PWR?
 U 1 1 61EA1AC2
 P 10000 3350
@@
 	6700 4700 6700 4600
 $Comp
-L IO_LINK_LIB:3V3_T2 #PWR?
+L IO_LINK-rescue:3V3_T2-IO_LINK_LIB #PWR?
 U 1 1 604C36E1
 P 6700 4600
@@
 	13650 5600 13650 5800
 $Comp
-L IO_LINK_LIB:SPT01-335DEE D?
+L IO_LINK-rescue:SPT01-335DEE-IO_LINK_LIB D?
 U 1 1 61EA17FF
 P 13750 5800
@@
 	14450 3950 14350 3950
 $Comp
-L IO_LINK_LIB:G #PWR?
+L IO_LINK-rescue:G-IO_LINK_LIB #PWR?
 U 1 1 61EA17EE
 P 14350 4900
@@
 $EndComp
 $Comp
-L IO_LINK_LIB:Screw_Terminal_01x04 J?
+L IO_LINK-rescue:Screw_Terminal_01x04-IO_LINK_LIB J?
 U 1 1 61EA17DC
 P 14650 3950
@@
 	12600 4050 12600 4400
 $Comp
-L IO_LINK_LIB:100nF_50V_0603 C?
+L IO_LINK-rescue:100nF_50V_0603-IO_LINK_LIB C?
 U 1 1 607068DF
 P 12150 4550
