File: pcb/IO_LINK_3.sch (KiCad schematic (older format))
At the start: 31 parts, among them J7 Screw_Terminal_01x04, U5 L6360TR

Commit message: PCB Release
Parts:
- C61, C62, C63, C64: symbol IO_LINK_LIB:22pF_50V_0603 -> IO_LINK-rescue:22pF_50V_0603-IO_LINK_LIB
- C65: symbol IO_LINK_LIB:2.2uF_16V_0603 -> IO_LINK-rescue:2.2uF_16V_0603-IO_LINK_LIB
- C66, C70, C72: symbol IO_LINK_LIB:100nF_25V_0603 -> IO_LINK-rescue:100nF_25V_0603-IO_LINK_LIB
- C67: symbol IO_LINK_LIB:10uF_50V_6.3mm_x_5.8mm_electrolytic -> IO_LINK-rescue:10uF_50V_6.3mm_x_5.8mm_electrolytic-IO_LINK_LIB
- C68, C69, C78: symbol IO_LINK_LIB:100nF_50V_0603 -> IO_LINK-rescue:100nF_50V_0603-IO_LINK_LIB
- C71: symbol IO_LINK_LIB:1uF_10V_0603 -> IO_LINK-rescue:1uF_10V_0603-IO_LINK_LIB
- C73, C74: symbol IO_LINK_LIB:560pF_50V_0603 -> IO_LINK-rescue:560pF_50V_0603-IO_LINK_LIB
- D19, D20: symbol IO_LINK_LIB:STPS1L40M -> IO_LINK-rescue:STPS1L40M-IO_LINK_LIB
- D21: symbol IO_LINK_LIB:LED_RED -> IO_LINK-rescue:LED_RED-IO_LINK_LIB
- D22: symbol IO_LINK_LIB:LED_GREEN -> IO_LINK-rescue:LED_GREEN-IO_LINK_LIB
- D23: symbol IO_LINK_LIB:SPT01-335DEE -> IO_LINK-rescue:SPT01-335DEE-IO_LINK_LIB
- J7: symbol IO_LINK_LIB:Screw_Terminal_01x04 -> IO_LINK-rescue:Screw_Terminal_01x04-IO_LINK_LIB
- R36, R37, R38, R39: symbol IO_LINK_LIB:10k_1%_0.1W_0603 -> IO_LINK-rescue:10k_1%_0.1W_0603-IO_LINK_LIB
- R40: symbol IO_LINK_LIB:124k_0.1%_0.1W_0603 -> IO_LINK-rescue:124k_0.1%_0.1W_0603-IO_LINK_LIB
- R41, R42: symbol IO_LINK_LIB:680R_1%_0.1W_0603 -> IO_LINK-rescue:680R_1%_0.1W_0603-IO_LINK_LIB
- R43: symbol IO_LINK_LIB:100R_1%_0.1W_0603 -> IO_LINK-rescue:100R_1%_0.1W_0603-IO_LINK_LIB
- R44: symbol IO_LINK_LIB:15R_1%_0.1W_0603 -> IO_LINK-rescue:15R_1%_0.1W_0603-IO_LINK_LIB
- U5: symbol IO_LINK_LIB:L6360TR -> IO_LINK-rescue:L6360TR-IO_LINK_LIB
Changed lines of the file:
@@
 EESchema Schematic File Version 4
+LIBS:IO_LINK-cache
 EELAYER 30 0
 EELAYER END
@@
 $EndDescr
 $Comp
-L IO_LINK_LIB:Screw_Terminal_01x04 J?
+L IO_LINK-rescue:Screw_Terminal_01x04-IO_LINK_LIB J?
 U 1 1 61EBCECE
 P 14650 3950
@@
 	9050 5600 9100 5600
 $Comp
-L IO_LINK_LIB:G #PWR?
+L IO_LINK-rescue:G-IO_LINK_LIB #PWR?
 U 1 1 61EBCEE0
 P 14350 4900
@@
 	14350 3950 14350 4900
 $Comp
-L IO_LINK_LIB:100R_1%_0.1W_0603 R?
+L IO_LINK-rescue:100R_1%_0.1W_0603-IO_LINK_LIB R?
 U 1 1 61EBCF14
 P 11450 4250
 AR Path="/602CF7CD/61EBCF14" Ref="R?"  Part="1"
 AR Path="/61EAA4CD/61EBCF14" Ref="R43"  Part="1"
+AR Path="/61EBCF14" Ref="R43"  Part="1"
 F 0 "R43" V 11350 4250 50  0000 C CNN
 F 1 "100R_1%_0.1W_0603" V 10910 4370 50  0001 C CNN
@@
 $EndComp
 $Comp
-L IO_LINK_LIB:15R_1%_0.1W_0603 R?
+L IO_LINK-rescue:15R_1%_0.1W_0603-IO_LINK_LIB R?
 U 1 1 61EBCF20
 P 11450 4500
@@
 $EndComp
 $Comp
-L IO_LINK_LIB:STPS1L40M D?
+L IO_LINK-rescue:STPS1L40M-IO_LINK_LIB D?
 U 1 1 61EBCF29
 P 10350 4550
@@
 $EndComp
 $Comp
-L IO_LINK_LIB:560pF_50V_0603 C?
+L IO_LINK-rescue:560pF_50V_0603-IO_LINK_LIB C?
 U 1 1 61EBCF34
 P 12600 4550
@@
 $EndComp
 $Comp
-L IO_LINK_LIB:10uF_50V_6.3mm_x_5.8mm_electrolytic C?
+L IO_LINK-rescue:10uF_50V_6.3mm_x_5.8mm_electrolytic-IO_LINK_LIB C?
 U 1 1 61EBCF3F
 P 7000 2150
@@
 $EndComp
 $Comp
-L IO_LINK_LIB:100nF_50V_0603 C?
+L IO_LINK-rescue:100nF_50V_0603-IO_LINK_LIB C?
 U 1 1 61EBCF4A
 P 7950 2150
@@
 	10350 4150 10350 4400
 $Comp
-L IO_LINK_LIB:STPS1L40M D?
+L IO_LINK-rescue:STPS1L40M-IO_LINK_LIB D?
 U 1 1 61EBCF68
 P 10700 4550
@@
 	13100 4700 13100 4900
 $Comp
-L IO_LINK_LIB:560pF_50V_0603 C?
+L IO_LINK-rescue:560pF_50V_0603-IO_LINK_LIB C?
 U 1 1 61EBCFA0
 P 13100 4550
@@
 	9800 4700 10000 4700
 $Comp
-L IO_LINK_LIB:680R_1%_0.1W_0603 R?
+L IO_LINK-rescue:680R_1%_0.1W_0603-IO_LINK_LIB R?
 U 1 1 61EBCFEA
 P 10600 5350
@@
 	10000 4700 10000 5350
 $Comp
-L IO_LINK_LIB:680R_1%_0.1W_0603 R?
+L IO_LINK-rescue:680R_1%_0.1W_0603-IO_LINK_LIB R?
 U 1 1 61EBCFF8
 P 10600 5650
@@
 $EndComp
 $Comp
-L IO_LINK_LIB:LED_RED D?
+L IO_LINK-rescue:LED_RED-IO_LINK_LIB D?
 U 1 1 61EBD002
 P 11500 5350
@@
 $EndComp
 $Comp
-L IO_LINK_LIB:LED_GREEN D?
+L IO_LINK-rescue:LED_GREEN-IO_LINK_LIB D?
 U 1 1 61EBD00C
 P 11500 5650
@@
 	11900 5500 12150 5500
 $Comp
-L IO_LINK_LIB:100nF_25V_0603 C?
+L IO_LINK-rescue:100nF_25V_0603-IO_LINK_LIB C?
 U 1 1 61EBD022
 P 10450 3500
@@
 	10000 3500 10300 3500
 $Comp
-L IO_LINK_LIB:100nF_25V_0603 C?
+L IO_LINK-rescue:100nF_25V_0603-IO_LINK_LIB C?
 U 1 1 61EBD039
 P 9750 2150
@@
 	9750 2300 9750 2500
 $Comp
-L IO_LINK_LIB:100nF_50V_0603 C?
+L IO_LINK-rescue:100nF_50V_0603-IO_LINK_LIB C?
 U 1 1 61EBD04B
 P 7450 2150
@@
 	7000 2300 7000 2500
 $Comp
-L IO_LINK_LIB:VCC #PWR?
+L IO_LINK-rescue:VCC-IO_LINK_LIB #PWR?
 U 1 1 61EBD068
 P 7300 1900
@@
 $EndComp
 $Comp
-L IO_LINK_LIB:VCC #PWR?
+L IO_LINK-rescue:VCC-IO_LINK_LIB #PWR?
 U 1 1 61EBD06E
 P 7800 1900
@@
 	7450 1950 7450 2000
 $Comp
-L IO_LINK_LIB:VCC #PWR?
+L IO_LINK-rescue:VCC-IO_LINK_LIB #PWR?
 U 1 1 61EBD07B
 P 7000 1900
@@
 	8600 1700 7450 1700
 $Comp
-L IO_LINK_LIB:2.2uF_16V_0603 C?
+L IO_LINK-rescue:2.2uF_16V_0603-IO_LINK_LIB C?
 U 1 1 61EBD08A
 P 5700 2150
@@
 $EndComp
 $Comp
-L IO_LINK_LIB:100nF_25V_0603 C?
+L IO_LINK-rescue:100nF_25V_0603-IO_LINK_LIB C?
 U 1 1 61EBD095
 P 6200 2150
@@
 Connection ~ 5700 1700
 $Comp
-L IO_LINK_LIB:8V #PWR?
+L IO_LINK-rescue:8V-IO_LINK_LIB #PWR?
 U 1 1 61EBD0B1
 P 5600 1650
@@
 	5600 1650 5600 1700
 $Comp
-L IO_LINK_LIB:1uF_10V_0603 C?
+L IO_LINK-rescue:1uF_10V_0603-IO_LINK_LIB C?
 U 1 1 61EBD0BD
 P 10250 2150
@@
 	4800 3500 7800 3500
 $Comp
-L IO_LINK_LIB:10k_1%_0.1W_0603 R?
+L IO_LINK-rescue:10k_1%_0.1W_0603-IO_LINK_LIB R?
 U 1 1 61EBD0D9
 P 4800 3050
@@
 	4800 3200 4800 3500
 $Comp
-L IO_LINK_LIB:10k_1%_0.1W_0603 R?
+L IO_LINK-rescue:10k_1%_0.1W_0603-IO_LINK_LIB R?
 U 1 1 61EBD0E6
 P 4300 3050
@@
 	4300 3600 4300 3200
 $Comp
-L IO_LINK_LIB:10k_1%_0.1W_0603 R?
+L IO_LINK-rescue:10k_1%_0.1W_0603-IO_LINK_LIB R?
 U 1 1 61EBD0F3
 P 3800 3050
@@
 	3800 3700 3800 3200
 $Comp
-L IO_LINK_LIB:10k_1%_0.1W_0603 R?
+L IO_LINK-rescue:10k_1%_0.1W_0603-IO_LINK_LIB R?
 U 1 1 61EBD100
 P 3300 3050
@@
 	3300 3800 3300 3200
 $Comp
-L IO_LINK_LIB:3V3 #PWR?
+L IO_LINK-rescue:3V3-IO_LINK_LIB #PWR?
 U 1 1 61EBD107
 P 3300 2700
@@
 $EndComp
 $Comp
-L IO_LINK_LIB:3V3 #PWR?
+L IO_LINK-rescue:3V3-IO_LINK_LIB #PWR?
 U 1 1 61EBD10D
 P 3800 2700
@@
 $EndComp
 $Comp
-L IO_LINK_LIB:3V3 #PWR?
+L IO_LINK-rescue:3V3-IO_LINK_LIB #PWR?
 U 1 1 61EBD113
 P 4300 2700
@@
 $EndComp
 $Comp
-L IO_LINK_LIB:3V3 #PWR?
+L IO_LINK-rescue:3V3-IO_LINK_LIB #PWR?
 U 1 1 61EBD119
 P 4800 2700
@@
 	3300 2700 3300 2900
 $Comp
-L IO_LINK_LIB:22pF_50V_0603 C?
+L IO_LINK-rescue:22pF_50V_0603-IO_LINK_LIB C?
 U 1 1 61EBD128
 P 3800 4250
@@
 $EndComp
 $Comp
-L IO_LINK_LIB:22pF_50V_0603 C?
+L IO_LINK-rescue:22pF_50V_0603-IO_LINK_LIB C?
 U 1 1 61EBD133
 P 4800 4250
@@
 $EndComp
 $Comp
-L IO_LINK_LIB:22pF_50V_0603 C?
+L IO_LINK-rescue:22pF_50V_0603-IO_LINK_LIB C?
 U 1 1 61EBD13E
 P 4300 4250
@@
 $EndComp
 $Comp
-L IO_LINK_LIB:22pF_50V_0603 C?
+L IO_LINK-rescue:22pF_50V_0603-IO_LINK_LIB C?
 U 1 1 61EBD149
 P 3300 4250
@@
 T3_UC_SIO
 $Comp
-L IO_LINK_LIB:124k_0.1%_0.1W_0603 R?
+L IO_LINK-rescue:124k_0.1%_0.1W_0603-IO_LINK_LIB R?
 U 1 1 61EBD18A
 P 8050 5600
@@
 IO-LINK TRANSCEIVER no. 3
 $Comp
-L IO_LINK_LIB:3V3_T3 #PWR?
+L IO_LINK-rescue:3V3_T3-IO_LINK_LIB #PWR?
 U 1 1 61EBD1A8
 P 10350 1650
@@
 $EndComp
 $Comp
-L IO_LINK_LIB:3V3_T3 #PWR?
+L IO_LINK-rescue:3V3_T3-IO_LINK_LIB #PWR?
 U 1 1 61EBD1AE
 P 10000 3350
@@
 $EndComp
 $Comp
-L IO_LINK_LIB:3V3_T3 #PWR?
+L IO_LINK-rescue:3V3_T3-IO_LINK_LIB #PWR?
 U 1 1 61EBD1B4
 P 12150 5400
@@
 Connection ~ 7600 4700
 $Comp
-L IO_LINK_LIB:3V3_T3 #PWR?
+L IO_LINK-rescue:3V3_T3-IO_LINK_LIB #PWR?
 U 1 1 604D45AD
 P 6700 4600
@@
 	12600 4050 12600 4400
 $Comp
-L IO_LINK_LIB:100nF_50V_0603 C?
+L IO_LINK-rescue:100nF_50V_0603-IO_LINK_LIB C?
 U 1 1 60741351
 P 12150 4550
@@
 $EndComp
 $Comp
-L IO_LINK_LIB:SPT01-335DEE D?
+L IO_LINK-rescue:SPT01-335DEE-IO_LINK_LIB D?
 U 1 1 61EBCEF1
 P 13750 5800
@@
 $EndComp
 $Comp
-L IO_LINK_LIB:L6360TR U?
+L IO_LINK-rescue:L6360TR-IO_LINK_LIB U?
 U 1 1 61EBCEC6
 P 8800 4150
