File: pcb/Microcontroller.sch (KiCad schematic (older format))
At the start: 32 parts, among them J2 USB_B_Mini, J3 STM_PROGRAMING_CONNECTOR, M1 W5500_ETHERNET_PCB_MODULE, SW1 Tactile_Switch, U1 STM32F072RBTx, Y1 CRYSTAL_16MHz_4PADS

Commit message: PCB Release
Parts:
- C1, C2, C7, C9: symbol IO_LINK_LIB:22pF_50V_0603 -> IO_LINK-rescue:22pF_50V_0603-IO_LINK_LIB
- C10, C12, C14, C3, C4, C6: symbol IO_LINK_LIB:100nF_25V_0603 -> IO_LINK-rescue:100nF_25V_0603-IO_LINK_LIB
- C11, C13, C15, C5, C8: symbol IO_LINK_LIB:2.2uF_10V_0603 -> IO_LINK-rescue:2.2uF_10V_0603-IO_LINK_LIB
- C16: symbol IO_LINK_LIB:10uF_25V_0805 -> IO_LINK-rescue:10uF_25V_0805-IO_LINK_LIB
- C17: symbol IO_LINK_LIB:4.7uF_10V_0603 -> IO_LINK-rescue:4.7uF_10V_0603-IO_LINK_LIB
- D3: symbol IO_LINK_LIB:USBLC6-2SC6Y -> IO_LINK-rescue:USBLC6-2SC6Y-IO_LINK_LIB
- J2: symbol IO_LINK_LIB:USB_B_Mini -> IO_LINK-rescue:USB_B_Mini-IO_LINK_LIB
- J3: symbol IO_LINK_LIB:STM_PROGRAMING_CONNECTOR -> IO_LINK-rescue:STM_PROGRAMING_CONNECTOR-IO_LINK_LIB
- JP1: symbol IO_LINK_LIB:SOLDERED_SELECTOR -> IO_LINK-rescue:SOLDERED_SELECTOR-IO_LINK_LIB
- L1: symbol IO_LINK_LIB:Coil_100uH_0805 -> IO_LINK-rescue:Coil_100uH_0805-IO_LINK_LIB
- L2: symbol IO_LINK_LIB:FB_30R@100MHz -> IO_LINK-rescue:FB_30R@100MHz-IO_LINK_LIB
- M1: symbol IO_LINK_LIB:W5500_ETHERNET_PCB_MODULE -> IO_LINK-rescue:W5500_ETHERNET_PCB_MODULE-IO_LINK_LIB
- R1, R2, R3: symbol IO_LINK_LIB:4k7_1%_0.1W_0603 -> IO_LINK-rescue:4k7_1%_0.1W_0603-IO_LINK_LIB
- R4: symbol IO_LINK_LIB:100R_1%_0.1W_0603 -> IO_LINK-rescue:100R_1%_0.1W_0603-IO_LINK_LIB
- R45: symbol IO_LINK_LIB:10k_1%_0.1W_0603 -> IO_LINK-rescue:10k_1%_0.1W_0603-IO_LINK_LIB
- SW1: symbol IO_LINK_LIB:Tactile_Switch -> IO_LINK-rescue:Tactile_Switch-IO_LINK_LIB
- Y1: symbol IO_LINK_LIB:CRYSTAL_16MHz_4PADS -> IO_LINK-rescue:CRYSTAL_16MHz_4PADS-IO_LINK_LIB
Changed lines of the file:
@@
 EESchema Schematic File Version 4
+LIBS:IO_LINK-cache
 EELAYER 30 0
 EELAYER END
@@
 $EndComp
 $Comp
-L IO_LINK_LIB:USB_B_Mini J?
+L IO_LINK-rescue:USB_B_Mini-IO_LINK_LIB J?
 U 1 1 61C677D4
 P 12650 1450
@@
 	13150 1650 13150 1850
 $Comp
-L IO_LINK_LIB:100R_1%_0.1W_0603 R?
+L IO_LINK-rescue:100R_1%_0.1W_0603-IO_LINK_LIB R?
 U 1 1 61C677E2
 P 13150 2000
 AR Path="/602BD8C8/61C677E2" Ref="R?"  Part="1"
 AR Path="/602BA3BC/61C677E2" Ref="R4"  Part="1"
+AR Path="/61C677E2" Ref="R4"  Part="1"
 F 0 "R4" H 13218 2182 50  0000 L CNN
 F 1 "100R_1%_0.1W_0603" V 12610 2120 50  0001 C CNN
@@
 $EndComp
 $Comp
-L IO_LINK_LIB:5V #PWR?
+L IO_LINK-rescue:5V-IO_LINK_LIB #PWR?
 U 1 1 61C677F7
 P 13150 1050
@@
 	16000 1500 16000 1050
 $Comp
-L IO_LINK_LIB:5V #PWR?
+L IO_LINK-rescue:5V-IO_LINK_LIB #PWR?
 U 1 1 61C6780A
 P 16000 1050
@@
 Connection ~ 12600 2300
 $Comp
-L IO_LINK_LIB:FB_30R@100MHz L?
+L IO_LINK-rescue:FB_30R@100MHz-IO_LINK_LIB L?
 U 1 1 61C6782E
 P 12550 2100
@@
 	12150 5400 17150 5400
 $Comp
-L IO_LINK_LIB:W5500_ETHERNET_PCB_MODULE M?
+L IO_LINK-rescue:W5500_ETHERNET_PCB_MODULE-IO_LINK_LIB M?
 U 1 1 61C59FFF
 P 14550 3850
@@
 	13850 4450 14100 4450
 $Comp
-L IO_LINK_LIB:4.7uF_10V_0603 C17
+L IO_LINK-rescue:4.7uF_10V_0603-IO_LINK_LIB C17
 U 1 1 61C84C68
 P 15800 3600
@@
 Connection ~ 15800 3300
 $Comp
-L IO_LINK_LIB:3V3 #PWR?
+L IO_LINK-rescue:3V3-IO_LINK_LIB #PWR?
 U 1 1 61D08B77
 P 16100 3250
@@
 SCL
 $Comp
-L IO_LINK_LIB:22pF_50V_0603 C7
+L IO_LINK-rescue:22pF_50V_0603-IO_LINK_LIB C7
 U 1 1 61F6D108
 P 7450 6000
@@
 $EndComp
 $Comp
-L IO_LINK_LIB:22pF_50V_0603 C9
+L IO_LINK-rescue:22pF_50V_0603-IO_LINK_LIB C9
 U 1 1 61F6DCDB
 P 7950 6000
@@
 $EndComp
 $Comp
-L IO_LINK_LIB:4k7_1%_0.1W_0603 R2
+L IO_LINK-rescue:4k7_1%_0.1W_0603-IO_LINK_LIB R2
 U 1 1 61F7ADE6
 P 7700 5250
@@
 $EndComp
 $Comp
-L IO_LINK_LIB:4k7_1%_0.1W_0603 R3
+L IO_LINK-rescue:4k7_1%_0.1W_0603-IO_LINK_LIB R3
 U 1 1 61F7C2E1
 P 8250 5250
@@
 	8250 5100 8250 4950
 $Comp
-L IO_LINK_LIB:3V3 #PWR?
+L IO_LINK-rescue:3V3-IO_LINK_LIB #PWR?
 U 1 1 61F83294
 P 7700 4950
@@
 $EndComp
 $Comp
-L IO_LINK_LIB:3V3 #PWR?
+L IO_LINK-rescue:3V3-IO_LINK_LIB #PWR?
 U 1 1 61F83FC5
 P 8250 4950
@@
 $EndComp
 $Comp
-L IO_LINK_LIB:CRYSTAL_16MHz_4PADS Y1
+L IO_LINK-rescue:CRYSTAL_16MHz_4PADS-IO_LINK_LIB Y1
 U 1 1 61F8644A
 P 2050 5100
@@
 $EndComp
 $Comp
-L IO_LINK_LIB:Tactile_Switch SW1
+L IO_LINK-rescue:Tactile_Switch-IO_LINK_LIB SW1
 U 1 1 61F883EF
 P 1650 3400
@@
 	2150 3300 1950 3300
 $Comp
-L IO_LINK_LIB:100nF_25V_0603 C3
+L IO_LINK-rescue:100nF_25V_0603-IO_LINK_LIB C3
 U 1 1 61F99A8F
 P 2550 3600
@@
 Connection ~ 2550 3300
 $Comp
-L IO_LINK_LIB:4k7_1%_0.1W_0603 R1
+L IO_LINK-rescue:4k7_1%_0.1W_0603-IO_LINK_LIB R1
 U 1 1 61FAB46B
 P 2550 2950
@@
 	2550 2800 2550 2600
 $Comp
-L IO_LINK_LIB:3V3 #PWR?
+L IO_LINK-rescue:3V3-IO_LINK_LIB #PWR?
 U 1 1 61FAFCF9
 P 2550 2600
@@
 SWCLK
 $Comp
-L IO_LINK_LIB:22pF_50V_0603 C2
+L IO_LINK-rescue:22pF_50V_0603-IO_LINK_LIB C2
 U 1 1 620705AC
 P 2500 5400
@@
 $EndComp
 $Comp
-L IO_LINK_LIB:22pF_50V_0603 C1
+L IO_LINK-rescue:22pF_50V_0603-IO_LINK_LIB C1
 U 1 1 62072211
 P 1600 5400
@@
 	5050 6900 5150 6900
 $Comp
-L IO_LINK_LIB:100nF_25V_0603 C4
+L IO_LINK-rescue:100nF_25V_0603-IO_LINK_LIB C4
 U 1 1 623C9E4B
 P 6050 2000
@@
 	6050 1650 5450 1650
 $Comp
-L IO_LINK_LIB:3V3 #PWR?
+L IO_LINK-rescue:3V3-IO_LINK_LIB #PWR?
 U 1 1 6243D6FF
 P 6650 1750
@@
 $EndComp
 $Comp
-L IO_LINK_LIB:10uF_25V_0805 C16
+L IO_LINK-rescue:10uF_25V_0805-IO_LINK_LIB C16
 U 1 1 624CF283
 P 11050 2000
@@
 	11050 2150 11050 2350
 $Comp
-L IO_LINK_LIB:3V3 #PWR?
+L IO_LINK-rescue:3V3-IO_LINK_LIB #PWR?
 U 1 1 624EC1F2
 P 11050 1250
@@
 	11050 1250 11050 1850
 $Comp
-L IO_LINK_LIB:3V3 #PWR?
+L IO_LINK-rescue:3V3-IO_LINK_LIB #PWR?
 U 1 1 624FAD5A
 P 4950 2950
@@
 $EndComp
 $Comp
-L IO_LINK_LIB:100nF_25V_0603 C6
+L IO_LINK-rescue:100nF_25V_0603-IO_LINK_LIB C6
 U 1 1 62509304
 P 7350 2000
@@
 $EndComp
 $Comp
-L IO_LINK_LIB:2.2uF_10V_0603 C5
+L IO_LINK-rescue:2.2uF_10V_0603-IO_LINK_LIB C5
 U 1 1 6252CBFA
 P 6500 2000
@@
 	6500 1800 6500 1850
 $Comp
-L IO_LINK_LIB:3V3 #PWR?
+L IO_LINK-rescue:3V3-IO_LINK_LIB #PWR?
 U 1 1 62566702
 P 7950 1750
@@
 $EndComp
 $Comp
-L IO_LINK_LIB:2.2uF_10V_0603 C8
+L IO_LINK-rescue:2.2uF_10V_0603-IO_LINK_LIB C8
 U 1 1 6256670D
 P 7800 2000
@@
 $EndComp
 $Comp
-L IO_LINK_LIB:100nF_25V_0603 C10
+L IO_LINK-rescue:100nF_25V_0603-IO_LINK_LIB C10
 U 1 1 625E7D9B
 P 8250 2000
@@
 $EndComp
 $Comp
-L IO_LINK_LIB:3V3 #PWR?
+L IO_LINK-rescue:3V3-IO_LINK_LIB #PWR?
 U 1 1 625E7DA1
 P 8850 1750
@@
 $EndComp
 $Comp
-L IO_LINK_LIB:2.2uF_10V_0603 C11
+L IO_LINK-rescue:2.2uF_10V_0603-IO_LINK_LIB C11
 U 1 1 625E7DAC
 P 8700 2000
@@
 $EndComp
 $Comp
-L IO_LINK_LIB:100nF_25V_0603 C12
+L IO_LINK-rescue:100nF_25V_0603-IO_LINK_LIB C12
 U 1 1 6263984E
 P 9150 2000
@@
 $EndComp
 $Comp
-L IO_LINK_LIB:3V3 #PWR?
+L IO_LINK-rescue:3V3-IO_LINK_LIB #PWR?
 U 1 1 62639854
 P 9750 1750
@@
 $EndComp
 $Comp
-L IO_LINK_LIB:2.2uF_10V_0603 C13
+L IO_LINK-rescue:2.2uF_10V_0603-IO_LINK_LIB C13
 U 1 1 6263985F
 P 9600 2000
@@
 $EndComp
 $Comp
-L IO_LINK_LIB:100nF_25V_0603 C14
+L IO_LINK-rescue:100nF_25V_0603-IO_LINK_LIB C14
 U 1 1 6269A4F8
 P 10100 2000
@@
 $EndComp
 $Comp
-L IO_LINK_LIB:3V3 #PWR?
+L IO_LINK-rescue:3V3-IO_LINK_LIB #PWR?
 U 1 1 6269A4FE
 P 10700 1750
@@
 $EndComp
 $Comp
-L IO_LINK_LIB:2.2uF_10V_0603 C15
+L IO_LINK-rescue:2.2uF_10V_0603-IO_LINK_LIB C15
 U 1 1 6269A509
 P 10550 2000
@@
 	10550 1250 10550 1800
 $Comp
-L IO_LINK_LIB:Coil_100uH_0805 L1
+L IO_LINK-rescue:Coil_100uH_0805-IO_LINK_LIB L1
 U 1 1 626CE77A
 P 7000 1550
@@
 $EndComp
 $Comp
-L IO_LINK_LIB:3V3 #PWR?
+L IO_LINK-rescue:3V3-IO_LINK_LIB #PWR?
 U 1 1 62882D06
 P 3750 3600
@@
 	3500 6100 4450 6100
 $Comp
-L IO_LINK_LIB:SOLDERED_SELECTOR JP1
+L IO_LINK-rescue:SOLDERED_SELECTOR-IO_LINK_LIB JP1
 U 1 1 62AC9BBF
 P 3500 3900
@@
 22.02.2021\n
 $Comp
-L IO_LINK_LIB:10k_1%_0.1W_0603 R45
+L IO_LINK-rescue:10k_1%_0.1W_0603-IO_LINK_LIB R45
 U 1 1 62B51CCF
 P 4200 3700
@@
 	4200 3900 4200 3850
 $Comp
-L IO_LINK_LIB:3V3 #PWR?
+L IO_LINK-rescue:3V3-IO_LINK_LIB #PWR?
 U 1 1 603CC200
 P 14600 6350
@@
 $EndComp
 $Comp
-L IO_LINK_LIB:STM_PROGRAMING_CONNECTOR J3
+L IO_LINK-rescue:STM_PROGRAMING_CONNECTOR-IO_LINK_LIB J3
 U 1 1 6049EB20
 P 14900 6900
@@
 	3500 6000 4450 6000
 $Comp
-L IO_LINK_LIB:USBLC6-2SC6Y D3
+L IO_LINK-rescue:USBLC6-2SC6Y-IO_LINK_LIB D3
 U 1 1 604A30DB
 P 14100 1400
