File: pcb/Power_Supply.sch (KiCad schematic (older format))
At the start: 13 parts, among them J1 Screw_Terminal_01x02, M2 DC_DC_CONVERTER_LM2596_PCB_MO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

Commit message: PCB Release
Parts:
- C18: symbol IO_LINK_LIB:15uF_16V_0805 -> IO_LINK-rescue:15uF_16V_0805-IO_LINK_LIB
- D1: symbol IO_LINK_LIB:SM15T33CAY -> IO_LINK-rescue:SM15T33CAY-IO_LINK_LIB
- D2: symbol IO_LINK_LIB:STPS1H100A -> IO_LINK-rescue:STPS1H100A-IO_LINK_LIB
- JP3: symbol IO_LINK_LIB:JUMPER_0805 -> IO_LINK-rescue:JUMPER_0805-IO_LINK_LIB
- M2: symbol IO_LINK_LIB:DC_DC_CONVERTER_LM2596_PCB_MODULE -> IO_LINK-rescue:DC_DC_CONVERTER_LM2596_PCB_MODULE-IO_LINK_LIB
- R5, R6, R7, R8: symbol IO_LINK_LIB:1R_1%_0.1W_0603 -> IO_LINK-rescue:1R_1%_0.1W_0603-IO_LINK_LIB
- TP1, TP2: symbol IO_LINK_LIB:TestPoint -> IO_LINK-rescue:TestPoint-IO_LINK_LIB
Changed lines of the file:
@@
 EESchema Schematic File Version 4
+LIBS:IO_LINK-cache
 EELAYER 30 0
 EELAYER END
@@
 POWER SUPPLY CONNECTOR AND PROTECTION CIRCUIT
 $Comp
-L IO_LINK_LIB:SM15T33CAY D1
+L IO_LINK-rescue:SM15T33CAY-IO_LINK_LIB D1
 U 1 1 603F2BFA
 P 1900 1650
@@
 	650  2300 5150 2300
 $Comp
-L IO_LINK_LIB:VCC #PWR0102
+L IO_LINK-rescue:VCC-IO_LINK_LIB #PWR0102
 U 1 1 604029F6
 P 3300 1150
@@
 	3300 1150 3300 1200
 $Comp
-L IO_LINK_LIB:VCC #PWR0103
+L IO_LINK-rescue:VCC-IO_LINK_LIB #PWR0103
 U 1 1 60404173
 P 1050 3050
@@
 	4550 3150 4650 3150
 $Comp
-L IO_LINK_LIB:TestPoint TP2
+L IO_LINK-rescue:TestPoint-IO_LINK_LIB TP2
 U 1 1 60467095
 P 4650 3050
@@
 Connection ~ 4650 3150
 $Comp
-L IO_LINK_LIB:TestPoint TP1
+L IO_LINK-rescue:TestPoint-IO_LINK_LIB TP1
 U 1 1 60468B85
 P 4150 3050
@@
 	4650 3150 4850 3150
 $Comp
-L IO_LINK_LIB:8V #PWR0147
+L IO_LINK-rescue:8V-IO_LINK_LIB #PWR0147
 U 1 1 6046D08A
 P 4850 3100
@@
 	1900 1200 3300 1200
 $Comp
-L IO_LINK_LIB:STPS1H100A D2
+L IO_LINK-rescue:STPS1H100A-IO_LINK_LIB D2
 U 1 1 603F8E2A
 P 2850 1900
@@
 DC-DC SMPS POWER SUPPLY SECTION
 $Comp
-L IO_LINK_LIB:DC_DC_CONVERTER_LM2596_PCB_MODULE M2
+L IO_LINK-rescue:DC_DC_CONVERTER_LM2596_PCB_MODULE-IO_LINK_LIB M2
 U 1 1 61B8D6D6
 P 1700 3250
@@
 Connection ~ 4150 3150
 $Comp
-L IO_LINK_LIB:15uF_16V_0805 C18
+L IO_LINK-rescue:15uF_16V_0805-IO_LINK_LIB C18
 U 1 1 60423361
 P 3550 3500
@@
 	650  2450 5150 2450
 $Comp
-L IO_LINK_LIB:3V3_T0 #PWR?
+L IO_LINK-rescue:3V3_T0-IO_LINK_LIB #PWR?
 U 1 1 61ECC7D2
 P 1200 5200
@@
 $EndComp
 $Comp
-L IO_LINK_LIB:3V3_T1 #PWR?
+L IO_LINK-rescue:3V3_T1-IO_LINK_LIB #PWR?
 U 1 1 61ECC7D8
 P 1200 5600
@@
 $EndComp
 $Comp
-L IO_LINK_LIB:3V3_T2 #PWR?
+L IO_LINK-rescue:3V3_T2-IO_LINK_LIB #PWR?
 U 1 1 61ECC7DE
 P 1200 6000
@@
 $EndComp
 $Comp
-L IO_LINK_LIB:3V3_T3 #PWR?
+L IO_LINK-rescue:3V3_T3-IO_LINK_LIB #PWR?
 U 1 1 61ECC7E4
 P 1200 6400
@@
 $EndComp
 $Comp
-L IO_LINK_LIB:1R_1%_0.1W_0603 R?
+L IO_LINK-rescue:1R_1%_0.1W_0603-IO_LINK_LIB R?
 U 1 1 61ECC7F0
 P 1750 6500
@@
 	2300 5700 2300 5300
 $Comp
-L IO_LINK_LIB:1R_1%_0.1W_0603 R?
+L IO_LINK-rescue:1R_1%_0.1W_0603-IO_LINK_LIB R?
 U 1 1 61ECC809
 P 1750 5300
@@
 $EndComp
 $Comp
-L IO_LINK_LIB:1R_1%_0.1W_0603 R?
+L IO_LINK-rescue:1R_1%_0.1W_0603-IO_LINK_LIB R?
 U 1 1 61ECC815
 P 1750 5700
@@
 	2300 5900 2300 6100
 $Comp
-L IO_LINK_LIB:1R_1%_0.1W_0603 R?
+L IO_LINK-rescue:1R_1%_0.1W_0603-IO_LINK_LIB R?
 U 1 1 61ECC825
 P 1750 6100
@@
 	2300 5900 2700 5900
 $Comp
-L IO_LINK_LIB:3V3 #PWR?
+L IO_LINK-rescue:3V3-IO_LINK_LIB #PWR?
 U 1 1 61ECC82F
 P 2700 5800
@@
 	650  4600 650  7050
 $Comp
-L IO_LINK_LIB:JUMPER_0805 JP3
+L IO_LINK-rescue:JUMPER_0805-IO_LINK_LIB JP3
 U 1 1 62B45572
 P 3700 1900
@@
 	4050 1900 4050 2050
 $Comp
-L IO_LINK_LIB:G #PWR?
+L IO_LINK-rescue:G-IO_LINK_LIB #PWR?
 U 1 1 62B49D15
 P 2850 4150
@@
 	2850 3900 2850 4150
 $Comp
-L IO_LINK_LIB:G #PWR?
+L IO_LINK-rescue:G-IO_LINK_LIB #PWR?
 U 1 1 62B4AEFC
 P 3550 4150
@@
 	3550 3650 3550 4150
 $Comp
-L IO_LINK_LIB:G #PWR?
+L IO_LINK-rescue:G-IO_LINK_LIB #PWR?
 U 1 1 62B4C6C8
 P 1050 4150
@@
 	1050 3900 1050 4150
 $Comp
-L IO_LINK_LIB:G #PWR?
+L IO_LINK-rescue:G-IO_LINK_LIB #PWR?
 U 1 1 62B4E619
 P 4050 2050
